Commit message: Update sample.urdf

File: Basics of pyBullet/Week 1/Subpart 2/sample.urdf (robot description, URDF)
Before this commit: robot r2d2, 11 links, 10 joints
Links:
- removed link box
- removed link head
- removed link left_back_wheel
- removed link left_base
- removed link left_front_wheel
- removed link left_leg
- removed link right_back_wheel
- removed link right_base
- removed link right_front_wheel
- added link right_leg1; visual box size=1 0.08 0.6
- link base_link: geometry visual cylinder length=0.6 radius=0.3
- link right_leg: geometry visual box size=1 0.075 0.6
Joints:
- removed joint base_to_left_leg
- removed joint head_swivel
- removed joint left_back_wheel_joint
- removed joint left_base_joint
- removed joint left_front_wheel_joint
- removed joint right_back_wheel_joint
- removed joint right_base_joint
- removed joint right_front_wheel_joint
- removed joint tobox
- added joint right_leg_to_right_leg1: type revolute, parent right_leg, child right_leg1, origin xyz=0.907 -0.907 0
- joint base_to_right_leg: origin xyz=0 -0.22 0.25 -> xyz=0 0 0; type fixed -> revolute
